File: 2_Schematics_and_Layout/0_Main_PDU/Main-DC-DC_Converter.kicad_sch (KiCad schematic)
At the start: 51 parts, among them U1 QSB40024S12, U2 1245HC100-RTR, U3 QSB40024S12

Commit message: Update
Other:
- note added: "% of load"
- note added: "10.81A"
- note added: "129.72W"
- note added: "14.57A"
- note added: "16.76A"
- note added: "17.25A"
- note added: "2"
- note added: "2.05"
- note added: "201.17W"
- note added: "21.62A"
- note added: "24V"
- note added: "259.44W"
- note added: "301.67W"
- note added: "33A"
- note added: "413.9W"
- note added: "42.23W dissipated as heat"
- note added: "481.28W"
- note added: "55.84%"
- note added: "67.38W dissipated as heat"
- note added: "67.9A"
- note added: "86.84%"
- note added: "="
- note added: "DC-DC η (efficiency) = 86%"
- note added: "Iin"
- note added: "Input Voltage (from battery) ="
- note added: "Max DC-DC Output Current"
- note added: "Max DC-DC Output Power and Current"
- note added: "Max Input Power and Current from Battery"
- note added: "Max PDU Output Current"
- note added: "Max PDU Output Power"
- note added: "Nominal DC-DC Output Power and Current"
- note added: "Nominal Input Power and Current from Battery"
- note added: "Nominal PDU Output Current"
- note added: "Nominal PDU Output Power"
- note added: "Output Current per Conv."
- note added: "Output Power per Conv."
- note added: "Output Voltage ="
- note added: "Required DC-DC Conv."
- note removed: "% of load ="
- note removed: "12.00V"
- note removed: "13.57A"
- note removed: "181.24W"
- note removed: "210.74W"
- note removed: "28.00V"
- note removed: "28V"
- note removed: "29.5W dissipated as heat"
- note removed: "326.9"
- note removed: "326.9W"
- note removed: "380.11W"
- note removed: "380.11w"
- note removed: "53.2W dissipated as heat"
- note removed: "7.53A"
- note removed: "86%"
- note removed: "= 15.1033A"
- note removed: "= 210.74W"
- note removed: "= 27.24A"
- note removed: "= 38.89%"
- note removed: "= 7.53A"
- note removed: "= 70.12%"
- note removed: "DC-DC Input Current Iin (full load) ="
- note removed: "DC-DC η (efficiency) ="
- note removed: "Iin ="
- note removed: "Iout ="
- note removed: "Maximum Input Current"
- note removed: "Maximum Output Current"
- note removed: "Maximum Output Power"
- note removed: "Minimum Input Current"
- note removed: "Minimum Output Current"
- note removed: "Minimum Output Power"
- note removed: "Pin ="
- note removed: "Total power output ="
- note removed: "Vin ="
- note removed: "Vout ="
- note removed: "______"
- note removed: "________"
- note removed: "_________"
- note removed: "____________________________________"
