File: 2_Schematics_and_Layout/5_COMMS_TELEM/14_COMMS_TELEM/Converter_DC-DC.kicad_sch (KiCad schematic)
At the start: 26 parts, among them U5 PDQ30-Q24-S5-D, U6 LT3080EST-PBF

Commit message: Update
Parts:
- U6: footprint SOT-3_ST_LIT -> Analog_Devices:SOT-3_ST_LIT
Changed lines of the file:
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@@
 			)
 		)
-		(property "Footprint" "SOT-3_ST_LIT"
+		(property "Footprint" "Analog_Devices:SOT-3_ST_LIT"
 			(at 121.666 108.712 0)
 			(effects
