File: 2_Schematics_and_Layout/5_COMMS_TELEM/14_COMMS_TELEM/LVDS_Enable_Drivers.kicad_sch (KiCad schematic)
At the start: 8 parts, among them U7 SN65LVDS387DGG, U8 DS90LV047ATMX/NOPB

Commit message: Update
Connections:
- net GNDT: no longer U8.7 (DIN4)
- net SPI_HV_SYNCn+: now reaches U8.10 (DOUT4+)
- net SPI_HV_SYNCn-: now reaches U8.9 (DOUT4-)
- removed net COLD_TPC_Charge_Pre-AMP_EN+: U7.40 (OUT4+_{B})
- net COLD_TPC_Charge_Pre-AMP_EN- renamed COLD_TPC_CHARGE_PREAMP_EN-
- net DAQ_CPU_EN renamed CPU_EN
- net DAQ_CPU_EN+ renamed CPU_EN+
- net DAQ_CPU_EN- renamed CPU_EN-
- new net COLD_TPC_CHARGE_PREAMP_EN+: U7.50 (OUT4+_{B})
- new net SPI_HV_SYNCn: U8.7 (DIN4)
- no-connect marks 2 -> 0
Other:
- moved on the sheet: U7B, U7C
