File: 2_Schematics_and_Layout/5_COMMS_TELEM/14_COMMS_TELEM/SiPM_VSET_DAQ.kicad_sch (KiCad schematic)
At the start: 84 parts, among them U19 LTC2050HVCS5-TRMPBF, U20 LTC2050HVCS5-TRMPBF, U21 DAC121S101CIMKX/NOPB, U22 DAC121S101CIMKX/NOPB, U23 LTC2050HVCS5-TRMPBF, U24 LTC2050HVCS5-TRMPBF, U25 DAC121S101CIMKX/NOPB, U26 DAC121S101CIMKX/NOPB, U27 LTC2050HVCS5-TRMPBF, U28 DAC121S101CIMKX/NOPB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

Commit message: Update
Parts:
- U19, U20, U23, U24, U27, U29: footprint S_5_ADI -> Analog_Devices:S_5_ADI
