File: 2_Schematics_and_Layout/6_WIRING_DIAGRAM/14_COMMS_TELEM.kicad_sch (KiCad schematic)
At the start: 16 parts, among them J14_1 618009231221, J14_10 1731130182, J14_11 618015330923, J14_12 618009231121, J14_13 1731130182, J14_14 618009231121, J14_16 Conn_01x09, J14_17 Conn_02x10_Odd_Even, J14_2 618025231221, J14_3 618025231221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

Commit message: Update
Parts:
- added J14_15: Conn_02x10_Odd_Even, Connector_PinHeader_2.54mm:PinHeader_2x12_P2.54mm_Vertical, symbol MSAG_Misc:Conn_02x12_Odd_Even
Connections:
- net SPI_CS_S4 is gone; now on net SPI_CS_S3: J14_17.24 (Pin_24)
- net GNDT: now also J14_15.10 (Pin_10), J14_15.15 (Pin_15), J14_15.20 (Pin_20), J14_15.5 (Pin_5)
- net SPI1_CS: now also J14_15.11 (Pin_11)
- net SPI1_DATA+: now also J14_15.2 (Pin_2)
- net SPI1_DATA-: now also J14_15.4 (Pin_4)
- net SPI1_DATA_IN: now also J14_15.9 (Pin_9)
- net SPI1_DATA_IN+: now also J14_15.6 (Pin_6)
- net SPI1_DATA_IN-: now also J14_15.8 (Pin_8)
- net SPI1_SCLK: now also J14_15.7 (Pin_7)
- net SPI1_SCLK+: now also J14_15.1 (Pin_1)
- net SPI1_SCLK-: now also J14_15.3 (Pin_3)
- net SPI_CS_S0: now also J14_17.21 (Pin_21); no longer J14_17.19 (Pin_19)
- net SPI_CS_S1: now also J14_17.22 (Pin_22); no longer J14_17.21 (Pin_21)
- net SPI_CS_S2: now also J14_17.23 (Pin_23); no longer J14_17.22 (Pin_22)
- net SPI_CS_S3: no longer J14_17.23 (Pin_23)
- new net TOF_BIAS_Enable: J14_17.19 (Pin_19)
Other:
- moved on the sheet: J14_10, J14_11, J14_12, J14_13, J14_9
