File: 2_Schematics_and_Layout/6_WIRING_DIAGRAM/6_WIRING_DIAGRAM.kicad_sch (KiCad schematic)
At the start: 43 parts

Commit message: Update
Parts:
- removed D1: LED, symbol Device:LED
Changed lines of the file:
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@@
 		)
 	)
-	(text "E"
-		(exclude_from_sim no)
-		(at 628.65 410.21 0)
-		(effects
-			(font
-				(size 3 3)
-				(thickness 0.6)
-				(bold yes)
-				(color 0 255 0 1)
-			)
-			(justify left)
-		)
-	)
 	(text "SMA"
 		(exclude_from_sim no)
@@
 		)
 	)
-	(text "L"
-		(exclude_from_sim no)
-		(at 626.11 410.21 0)
-		(effects
-			(font
-				(size 3 3)
-				(thickness 0.6)
-				(bold yes)
-				(color 255 0 0 1)
-			)
-			(justify left)
-		)
-	)
 	(text "Secondary PWR"
 		(exclude_from_sim no)
@@
 		)
 	)
-	(text "J5"
-		(exclude_from_sim no)
-		(at 231.14 292.1 0)
-		(effects
-			(font
-				(size 1.5 1.5)
-				(thickness 0.254)
-				(bold yes)
-			)
-		)
-	)
 	(text "J6  9-FDSUB"
 		(exclude_from_sim no)
@@
 		)
 	)
+	(text "J4"
+		(exclude_from_sim no)
+		(at 232.283 284.988 0)
+		(effects
+			(font
+				(size 1.5 1.5)
+				(thickness 0.254)
+				(bold yes)
+			)
+		)
+	)
 	(text "PMT"
 		(exclude_from_sim no)
@@
 		)
 	)
-	(text "SMA"
-		(exclude_from_sim no)
-		(at 228.6 284.48 0)
-		(effects
-			(font
-				(size 1.5 1.5)
-				(thickness 0.254)
-				(bold yes)
-			)
-			(justify right)
-		)
-	)
 	(text "W-205\n/\n9"
 		(exclude_from_sim no)
@@
 		)
 	)
-	(text "D"
-		(exclude_from_sim no)
-		(at 631.19 410.21 0)
-		(effects
-			(font
-				(size 3 3)
-				(thickness 0.6)
-				(bold yes)
-				(color 0 0 255 1)
-			)
-			(justify left)
-		)
-	)
 	(text "9-FDSUB"
 		(exclude_from_sim no)
@@
 		)
 	)
+	(text "J5"
+		(exclude_from_sim no)
+		(at 232.283 292.608 0)
+		(effects
+			(font
+				(size 1.5 1.5)
+				(thickness 0.254)
+				(bold yes)
+			)
+		)
+	)
 	(text "J14\n\n\n"
 		(exclude_from_sim no)
@@
 		)
 	)
-	(text "SMA"
-		(exclude_from_sim no)
-		(at 228.6 292.1 0)
-		(effects
-			(font
-				(size 1.5 1.5)
-				(thickness 0.254)
-				(bold yes)
-			)
-			(justify right)
-		)
-	)
 	(text "25-DSUB M-F:"
 		(exclude_from_sim no)
@@
 		)
 	)
+	(text "9-FDSUB"
+		(exclude_from_sim no)
+		(at 229.743 292.608 0)
+		(effects
+			(font
+				(size 1.5 1.5)
+				(thickness 0.254)
+				(bold yes)
+			)
+			(justify right)
+		)
+	)
 	(text "J10  9-FDSUB"
 		(exclude_from_sim no)
@@
 		)
 	)
-	(text "J4"
-		(exclude_from_sim no)
-		(at 231.14 284.48 0)
-		(effects
-			(font
-				(size 1.5 1.5)
-				(thickness 0.254)
-				(bold yes)
-			)
-		)
-	)
 	(text "+5V EN"
 		(exclude_from_sim no)
@@
 		)
 	)
+	(text "9-FDSUB"
+		(exclude_from_sim no)
+		(at 229.743 284.988 0)
+		(effects
+			(font
+				(size 1.5 1.5)
+				(thickness 0.254)
+				(bold yes)
+			)
+			(justify right)
+		)
+	)
 	(text "PMT"
 		(exclude_from_sim no)
@@
 		)
 	)
-	(wire
-		(pts
-			(xy 612.14 398.78) (xy 629.92 398.78)
-		)
-		(stroke
-			(width 0)
-			(type default)
-		)
-	)
 	(bus
 		(pts
@@
 		)
 	)
+	(wire
+		(pts
+			(xy 233.68 294.64) (xy 246.38 294.64)
+		)
+		(stroke
+			(width 0)
+			(type default)
+			(color 4 72 255 1)
+		)
+	)
 	(bus
 		(pts
@@
 		)
 	)
-	(wire
-		(pts
-			(xy 246.38 294.64) (xy 254 294.64)
-		)
-		(stroke
-			(width 1)
-			(type default)
-		)
-	)
 	(bus
 		(pts
@@
 	(wire
 		(pts
-			(xy 233.68 294.64) (xy 246.38 294.64)
-		)
-		(stroke
-			(width 0)
-			(type default)
-		)
-	)
-	(wire
-		(pts
 			(xy 200.66 208.28) (xy 200.66 200.66)
 		)
@@
 	(wire
 		(pts
-			(xy 204.47 304.8) (xy 204.47 311.15)
+			(xy 233.68 287.02) (xy 246.38 287.02)
 		)
 		(stroke
 			(width 0)
 			(type default)
+			(color 4 72 255 1)
 		)
 	)
-	(bus
+	(wire
 		(pts
-			(xy 243.84 469.9) (xy 246.38 469.9)
+			(xy 204.47 304.8) (xy 204.47 311.15)
 		)
 		(stroke
 			(width 0)
 			(type default)
-			(color 255 127 0 1)
 		)
 	)
-	(wire
+	(bus
 		(pts
-			(xy 246.38 287.02) (xy 254 287.02)
+			(xy 243.84 469.9) (xy 246.38 469.9)
 		)
 		(stroke
-			(width 1)
+			(width 0)
 			(type default)
+			(color 255 127 0 1)
 		)
 	)
@@
 	(wire
 		(pts
+			(xy 246.38 294.64) (xy 254 294.64)
+		)
+		(stroke
+			(width 1)
+			(type default)
+			(color 4 72 255 1)
+		)
+	)
+	(wire
+		(pts
 			(xy 419.1 134.62) (xy 424.18 134.62)
 		)
@@
 		)
 	)
-	(wire
-		(pts
-			(xy 612.14 406.4) (xy 629.92 406.4)
-		)
-		(stroke
-			(width 0)
-			(type default)
-		)
-	)
 	(bus
 		(pts
@@
 	(wire
 		(pts
+			(xy 246.38 287.02) (xy 254 287.02)
+		)
+		(stroke
+			(width 1)
+			(type default)
+			(color 4 72 255 1)
+		)
+	)
+	(wire
+		(pts
 			(xy 621.03 189.23) (xy 628.65 189.23)
 		)
@@
 	(wire
 		(pts
-			(xy 233.68 287.02) (xy 246.38 287.02)
-		)
-		(stroke
-			(width 0)
-			(type default)
-		)
-	)
-	(wire
-		(pts
 			(xy 403.86 124.46) (xy 419.1 124.46)
 		)
@@
 		)
 	)
-	(symbol
-		(lib_id "Device:LED")
-		(at 629.92 402.59 90)
-		(unit 1)
-		(exclude_from_sim no)
-		(in_bom yes)
-		(on_board yes)
-		(dnp no)
-		(fields_autoplaced yes)
-		(property "Reference" "D1"
-			(at 633.73 402.9074 90)
-			(effects
-				(font
-					(size 1.27 1.27)
-				)
-				(justify right)
-			)
-		)
-		(property "Value" "LED"
-			(at 633.73 405.4474 90)
-			(effects
-				(font
-					(size 1.27 1.27)
-				)
-				(justify right)
-			)
-		)
-		(property "Footprint" ""
-			(at 629.92 402.59 0)
-			(effects
-				(font
-					(size 1.27 1.27)
-				)
-				(hide yes)
-			)
-		)
-		(property "Datasheet" "~"
-			(at 629.92 402.59 0)
-			(effects
-				(font
-					(size 1.27 1.27)
-				)
-				(hide yes)
-			)
-		)
-		(property "Description" "Light emitting diode"
-			(at 629.92 402.59 0)
-			(effects
-				(font
-					(size 1.27 1.27)
-				)
-				(hide yes)
-			)
-		)
-		(pin "1"
-		)
-		(pin "2"
-		)
-		(instances
-			(project ""
-				(path "/99d2acbf-9222-44b4-9cd1-53dce752648e"
-					(reference "D1")
-					(unit 1)
-				)
-			)
-		)
-	)
